Commit message: Initial Commit

File: robotiq_description/urdf/robotiq_85_gripper.transmission.xacro (robot description, xacro)
@@ -5,11 +5,9 @@
       <type>transmission_interface/SimpleTransmission</type>
       <joint name="${prefix}robotiq_85_left_knuckle_joint">
-        <hardwareInterface>PositionJointInterface</hardwareInterface>
-        <!-- <hardwareInterface>EffortJointInterface</hardwareInterface> -->
+        <hardwareInterface>hardware_interface/PositionJointInterface</hardwareInterface>
       </joint>
       <actuator name="${prefix}robotiq_85_left_knuckle_motor">
         <mechanicalReduction>1</mechanicalReduction>
-        <hardwareInterface>PositionJointInterface</hardwareInterface>
-        <!-- <hardwareInterface>EfforJointInterface</hardwareInterface> -->
+        <hardwareInterface>hardware_interface/PositionJointInterface</hardwareInterface>
       </actuator>
     </transmission>

File: robotiq_description/urdf/robotiq_85_gripper.urdf.xacro (robot description, xacro)
@@ -33,4 +33,5 @@
       <origin rpy="${pi} 0.0 0.0" xyz="0.05490451627 0.03060114443 0.0"/>
       <limit lower="0.0" upper="0.80285" velocity="0.5" effort="1000"/>
+     <!-- <limit lower="-3.14" upper="3.14" velocity="100" effort="1000"/> -->
     </joint>
     <joint name="${prefix}robotiq_85_right_knuckle_joint" type="continuous">
@@ -39,5 +40,6 @@
       <axis xyz="0 0 1"/>
       <origin rpy="0.0 0.0 0.0" xyz="0.05490451627 -0.03060114443 0.0"/>
-      <limit lower="-3.14" upper="3.14" velocity="100.0" effort="1000"/>
+      <!-- <limit lower="-3.14" upper="3.14" velocity="100.0" effort="1000"/> -->
+      <limit lower="0.0" upper="0.80285" velocity="0.5" effort="1000"/>
       <mimic joint="${prefix}robotiq_85_left_knuckle_joint"/>
     </joint>
